File: Clavier75.kicad_sch (KiCad schematic)
At the start: 16 parts

Commit message: hehehehehehe
Parts:
- added D1, D2, D3, D4, D5: SOD-123, Diode_SMD:D_SOD-123, symbol Device:D_Small
- added MX1, MX3, MX4, MX5: MX-NoLED, MX_Alps_Hybrid:MX-1U, symbol MX_Alps_Hybrid:MX-NoLED
- C1, C2, C3, C4, C5, C6, C7: renamed from C?; footprint (none) -> Capacitor_SMD:C_0805_2012Metric
- F1: renamed from F?; footprint (none) -> Fuse:Fuse_1206_3216Metric
- R1, R2, R3, R4: renamed from R?; footprint (none) -> Resistor_SMD:R_0805_2012Metric
- gave numbers to parts that had none: 4
Connections:
- net ROW0: now reaches U1.27 (PD7)
- net ROW0: now also D1.1 (K), D2.1 (K), D4.1 (K)
- net COL1: now reaches U1.28 (PB4)
- net COL1: now also MX4.1 (COL), MX5.1 (COL)
- net COL0: now reaches U1.29 (PB5)
- net COL0: now also MX1.1 (COL), MX3.1 (COL)
- net ROW1: now reaches U1.30 (PB6)
- net ROW1: now also D3.1 (K), D5.1 (K)
- new net: D1.2 (A), D2.2 (A), MX1.2 (ROW)
- new net: D5.2 (A), MX5.2 (ROW)
- new net: D3.2 (A), MX3.2 (ROW)
- new net: D4.2 (A), MX4.2 (ROW)
Other:
- moved on the sheet: F1, USB1

Commit message: googoogaga
Parts:
- removed D1: SOD-123, Diode_SMD:D_SOD-123, symbol Device:D_Small
- SW1: footprint (none) -> KBParts:SKQG-1155865
- USB1: footprint (none) -> KBParts:Molex-0548190589
- Y1: footprint (none) -> Crystal:Crystal_SMD_3225-4Pin_3.2x2.5mm
Changed lines of the file:
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@@
   (junction (at 90.17 46.99) (diameter 0) (color 0 0 0 0)
-  )
-  (junction (at 217.17 87.63) (diameter 0) (color 0 0 0 0)
   )
   (junction (at 71.12 93.98) (diameter 0) (color 0 0 0 0)
@@
     (pin "1")
   )
-  (symbol (lib_id "Device:D_Small") (at 217.17 90.17 90) (unit 1)
-    (in_bom yes) (on_board yes) (fields_autoplaced)
-    (property "Reference" "D1" (id 0) (at 219.71 88.8999 90)
-      (effects (font (size 1.27 1.27)) (justify right))
-    )
-    (property "Value" "SOD-123" (id 1) (at 219.71 91.4399 90)
-      (effects (font (size 1.27 1.27)) (justify right))
-    )
-    (property "Footprint" "Diode_SMD:D_SOD-123" (id 2) (at 217.17 90.17 90)
-      (effects (font (size 1.27 1.27)) hide)
-    )
-    (property "Datasheet" "~" (id 3) (at 217.17 90.17 90)
-      (effects (font (size 1.27 1.27)) hide)
-    )
-    (pin "1")
-    (pin "2")
-  )
   (symbol (lib_id "Device:R") (at 153.67 90.17 90) (unit 1)
     (in_bom yes) (on_board yes) (fields_autoplaced)
@@
     (property "Reference" "Y1" (id 0) (at 104.14 38.9888 90))
     (property "Value" "16MHz" (id 1) (at 104.14 41.5288 90))
-    (property "Footprint" "" (id 2) (at 90.17 44.45 0)
+    (property "Footprint" "Crystal:Crystal_SMD_3225-4Pin_3.2x2.5mm" (id 2) (at 90.17 44.45 0)
       (effects (font (size 1.27 1.27)) hide)
     )
@@
     (property "Reference" "SW1" (id 0) (at 93.98 29.21 0))
     (property "Value" "SW_Push" (id 1) (at 93.98 31.75 0))
-    (property "Footprint" "" (id 2) (at 93.98 31.75 0)
+    (property "Footprint" "KBParts:SKQG-1155865" (id 2) (at 93.98 31.75 0)
       (effects (font (size 1.27 1.27)) hide)
     )
@@
   )
   (symbol (lib_id "Device:D_Small") (at 217.17 90.17 90) (unit 1)
-    (in_bom yes) (on_board yes) (fields_autoplaced)
+    (in_bom yes) (on_board yes)
     (property "Reference" "D2" (id 0) (at 219.71 88.8999 90)
       (effects (font (size 1.27 1.27)) (justify right))
@@
       (effects (font (size 1.524 1.524)))
     )
-    (property "Footprint" "" (id 2) (at 187.96 35.56 0)
+    (property "Footprint" "KBParts:Molex-0548190589" (id 2) (at 187.96 35.56 0)
       (effects (font (size 1.524 1.524)) hide)
     )
@@
       (reference "C7") (unit 1) (value "1uF") (footprint "Capacitor_SMD:C_0805_2012Metric")
     )
-    (path "/38f1a477-c484-4281-b958-d0c0cbdac2ac"
-      (reference "D1") (unit 1) (value "SOD-123") (footprint "Diode_SMD:D_SOD-123")
-    )
     (path "/dacda25b-a1d2-4165-ab12-0f5e1db6aa2d"
       (reference "D2") (unit 1) (value "SOD-123") (footprint "Diode_SMD:D_SOD-123")
@@
     )
     (path "/8c611282-6de6-435a-88a0-872567166b36"
-      (reference "SW1") (unit 1) (value "SW_Push") (footprint "")
+      (reference "SW1") (unit 1) (value "SW_Push") (footprint "KBParts:SKQG-1155865")
     )
     (path "/9d044540-5638-4cc7-8674-8264ab86206f"
@@
     )
     (path "/db828a5b-73df-4513-a6ea-10f05f33c89e"
-      (reference "USB1") (unit 1) (value "Molex-0548190589") (footprint "")
+      (reference "USB1") (unit 1) (value "Molex-0548190589") (footprint "KBParts:Molex-0548190589")
     )
     (path "/6f5a839b-afe6-472a-a8a6-493c6e6ffa21"
-      (reference "Y1") (unit 1) (value "16MHz") (footprint "")
-    )
-  )
+      (reference "Y1") (unit 1) (value "16MHz") (footprint "Crystal:Crystal_SMD_3225-4Pin_3.2x2.5mm")
+    )
+  )
