File: _autosave-Clavier75.kicad_pcb (KiCad board)
At the start: 2 copper layers, 25 parts, among them SW1 SW_Push, U1 ATmega32U4-A, Y1 16MHz

Commit message: googoogaga
Parts:
- removed D1: SOD-123, Diode_SMD:D_SOD-123
- moved D4 131.8 mm to (252.6, 123.9)
- moved D2 131.6 mm to (233.5, 123.8)
- moved MX1 131.6 mm to (225.3, 123.8)
- moved MX3 131.6 mm to (225.3, 142.9)
- moved MX4 131.6 mm to (244.3, 123.8)
- moved MX5 131.6 mm to (244.3, 142.9)
- moved R3 71.1 mm to (194.3, 145.0)
- moved D5 70.0 mm to (252.7, 142.8), turned to 90 degrees
- moved D3 59.0 mm to (233.6, 142.8), turned to 90 degrees
- moved C2 57.7 mm to (193.4, 132.0), turned to -90 degrees
- moved C6 57.7 mm to (208.4, 144.8)
- moved R2 56.0 mm to (183.0, 125.9), turned to 90 degrees
- moved SW1 54.8 mm to (184.4, 146.6)
- moved U1 52.8 mm to (203.2, 135.5), turned to 180 degrees
- moved C5 48.0 mm to (208.7, 122.1), turned to 90 degrees
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Other:
- board outline added: 76 x 38.3 mm
