File: Clavier75.kicad_pcb (KiCad board)
At the start: 2 copper layers, 25 parts, among them SW1 SW_Push, U1 ATmega32U4-A, Y1 16MHz

Commit message: rsdfsdfsdffsdfdsfss
Parts:
- removed D1: SOD-123, Diode_SMD:D_SOD-123
- USB1: moved to B.Cu
- moved D4 131.8 mm to (252.6, 123.9)
- moved D2 131.6 mm to (233.5, 123.8)
- moved MX1 131.6 mm to (225.3, 123.8)
- moved MX3 131.6 mm to (225.3, 142.9)
- moved MX4 131.6 mm to (244.3, 123.8)
- moved MX5 131.6 mm to (244.3, 142.9)
- moved C5 71.2 mm to (210.8, 146.8), turned to -90 degrees
- moved D5 70.0 mm to (252.7, 142.8), turned to 90 degrees
- moved D3 59.0 mm to (233.6, 142.8), turned to 90 degrees
- moved C2 55.0 mm to (213.6, 135.2), turned to 90 degrees
- moved SW1 54.8 mm to (184.4, 146.6)
- moved R2 54.8 mm to (184.2, 125.2), turned to -90 degrees
- moved C4 53.7 mm to (201.2, 146.8), turned to -90 degrees
- moved R4 52.9 mm to (192.1, 146.4), turned to 180 degrees
- moved C3 49.8 mm to (192.5, 137.5), turned to 180 degrees
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Routing:
- net Net-(R3-Pad2): track 0.00 -> 64.7 mm, vias 0 -> 3
- net +5V: track 0.00 -> 49.7 mm
- net GND: track 0.00 -> 40.3 mm
- net /ROW1: track 0.00 -> 19.7 mm
- net /ROW0: track 0.00 -> 19.6 mm
- net VCC: track 0.00 -> 18.3 mm, vias 0 -> 1
- net /COL1: track 0.00 -> 18.1 mm
- net /COL0: track 0.00 -> 18.1 mm
- net Net-(C4-Pad2): track 0.00 -> 17.5 mm
- net Net-(C4-Pad1): track 0.00 -> 10.3 mm
- net Net-(D1-Pad2): track 0.00 -> 8.20 mm
- net Net-(D5-Pad2): track 0.00 -> 8.06 mm
- net Net-(D4-Pad2): track 0.00 -> 7.90 mm
- net Net-(D3-Pad2): track 0.00 -> 7.61 mm
- net /D+: track 0.00 -> 4.01 mm
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Other:
- board outline added: 76 x 38.3 mm
